File: hardware/Drivers_Motores_ArduinoNANO/Drivers_Motores_ArduinoNANO.kicad_sch (KiCad schematic)
At the start: 25 parts, among them J2 V+-, J3 FTDI, J3 RS485, P2 HEADER_02X05, P3 HEADER_02X05, U1 AMS1117-5.0, U2 ATMEGA328P-AU, Y1 16MHz

Commit message: Nuevo PCb
Parts:
- removed C3: 100nF, Capacitor_SMD:C_0805_2012Metric_Pad1.18x1.45mm_HandSolder, symbol Device:C
- removed C3 (x2): 1uF, Capacitor_SMD:C_0805_2012Metric_Pad1.18x1.45mm_HandSolder, symbol Device:C
- removed C3: 4,7uF, Capacitor_SMD:C_0805_2012Metric_Pad1.18x1.45mm_HandSolder, symbol Device:C
- removed EN1: SW_Push, Button_Switch_THT:SW_PUSH_6mm_H5mm, symbol EESTN5:SW_Push
- removed J3: FTDI, Connector_PinHeader_2.54mm:PinHeader_1x04_P2.54mm_Horizontal, symbol Connector:Conn_01x04_Pin
- removed R2 (x2): 1K, EESTN5-v2:R_1206, symbol EESTN5:R
- removed R2: 10K, EESTN5-v2:R_1206, symbol EESTN5:R
- removed U2: ATMEGA328P-AU, EESTN5-v2:TQFP-32_7x7mm_Pitch0.8mm, symbol EESTN5-v2:ATMEGA328P-AU
- removed Y1: 16MHz, Crystal:Resonator_SMD_Murata_CSTxExxV-3Pin_3.0x1.1mm_HandSoldering, symbol Device:Resonator
- added J10, J11, J2, J5, J6, J7, J8, J9: Conn, Connector_PinHeader_2.54mm:PinHeader_1x03_P2.54mm_Vertical, symbol Sensor_Linea_Bonaerenses-rescue:Conn_01X03
- added J4: Arduino_Nano_Header, EESTN5-v2:arduino_nano_header, symbol EESTN5-v2:Arduino_Nano_Header
Connections:
- net +5V: now also J10.2 (P2), J11.2 (P2), J2.2 (P2), J4.27 (5V), J5.2 (P2), J6.2 (P2), J7.2 (P2), J8.2 (P2), J9.2 (P2)
- net DERE: now also J4.16 (SCK/D13)
- net GND: now also J10.3 (P3), J11.3 (P3), J2.3 (P3), J4.29 (GND), J4.4 (GND), J5.3 (P3), J6.3 (P3), J7.3 (P3), J8.3 (P3), J9.3 (P3)
- net LED_1: now also J4.11 (D8/ICP)
- net LED_2: now also J4.10 (D7/AIN1)
- net M1A: now also J4.13 (D10/SS)
- net M1B: now also J4.14 (D11/MOSI)
- net M2A: now also J4.8 (D5/T1)
- net M2B: now also J4.9 (D6/AIN0)
- net Rx: now also J4.2 (D0/RX)
- net Tx: now also J4.1 (D1/TX)
- new net 1: J2.1 (P1), J4.19 (A0)
- new net 2: J4.20 (A1), J5.1 (P1)
- new net 3: J4.21 (A2), J6.1 (P1)
- new net 4: J10.1 (P1), J4.22 (A3)
- new net 5: J4.23 (A4), J7.1 (P1)
- new net 6: J4.24 (A5), J8.1 (P1)
- new net 7: J4.25 (A6), J9.1 (P1)
- new net 8: J11.1 (P1), J4.26 (A7)
Other:
- note removed: "PROGRAMADOR"
- moved on the sheet: H1, H2, J3
